File: hardware/matrix.sch (KiCad schematic (older format))
At the start: 26 parts, among them P1 MATRIX_BOT, P2 MATRIX_TOP

Commit message: Fix silkscreen
Parts:
- R1, R10, R11, R12, R13, R14, R15, R16, R17, R18, R19, R2, R20, R21, R22, R23, R24, R3, R4, R5, R6, R7, R8, R9: footprint Resistors_SMD:R_0805 -> rgb-matrix:R_0805
Changed lines of the file:
@@
 F 0 "R12" V 4980 4400 50  0000 C CNN
 F 1 "100" V 4900 4400 50  0000 C CNN
-F 2 "Resistors_SMD:R_0805" V 4830 4400 50  0001 C CNN
+F 2 "rgb-matrix:R_0805" V 4830 4400 50  0001 C CNN
 F 3 "" H 4900 4400 50  0000 C CNN
 	1    4900 4400
@@
 F 0 "R1" V 4980 2900 50  0000 C CNN
 F 1 "100" V 4900 2900 50  0000 C CNN
-F 2 "Resistors_SMD:R_0805" V 4830 2900 50  0001 C CNN
+F 2 "rgb-matrix:R_0805" V 4830 2900 50  0001 C CNN
 F 3 "" H 4900 2900 50  0000 C CNN
 	1    4900 2900
@@
 F 0 "R2" V 4980 3000 50  0000 C CNN
 F 1 "100" V 4900 3000 50  0000 C CNN
-F 2 "Resistors_SMD:R_0805" V 4830 3000 50  0001 C CNN
+F 2 "rgb-matrix:R_0805" V 4830 3000 50  0001 C CNN
 F 3 "" H 4900 3000 50  0000 C CNN
 	1    4900 3000
@@
 F 0 "R3" V 4980 3100 50  0000 C CNN
 F 1 "100" V 4900 3100 50  0000 C CNN
-F 2 "Resistors_SMD:R_0805" V 4830 3100 50  0001 C CNN
+F 2 "rgb-matrix:R_0805" V 4830 3100 50  0001 C CNN
 F 3 "" H 4900 3100 50  0000 C CNN
 	1    4900 3100
@@
 F 0 "R4" V 4980 3200 50  0000 C CNN
 F 1 "100" V 4900 3200 50  0000 C CNN
-F 2 "Resistors_SMD:R_0805" V 4830 3200 50  0001 C CNN
+F 2 "rgb-matrix:R_0805" V 4830 3200 50  0001 C CNN
 F 3 "" H 4900 3200 50  0000 C CNN
 	1    4900 3200
@@
 F 0 "R5" V 4980 3300 50  0000 C CNN
 F 1 "100" V 4900 3300 50  0000 C CNN
-F 2 "Resistors_SMD:R_0805" V 4830 3300 50  0001 C CNN
+F 2 "rgb-matrix:R_0805" V 4830 3300 50  0001 C CNN
 F 3 "" H 4900 3300 50  0000 C CNN
 	1    4900 3300
@@
 F 0 "R6" V 4980 3400 50  0000 C CNN
 F 1 "100" V 4900 3400 50  0000 C CNN
-F 2 "Resistors_SMD:R_0805" V 4830 3400 50  0001 C CNN
+F 2 "rgb-matrix:R_0805" V 4830 3400 50  0001 C CNN
 F 3 "" H 4900 3400 50  0000 C CNN
 	1    4900 3400
@@
 F 0 "R11" V 4980 4300 50  0000 C CNN
 F 1 "100" V 4900 4300 50  0000 C CNN
-F 2 "Resistors_SMD:R_0805" V 4830 4300 50  0001 C CNN
+F 2 "rgb-matrix:R_0805" V 4830 4300 50  0001 C CNN
 F 3 "" H 4900 4300 50  0000 C CNN
 	1    4900 4300
@@
 F 0 "R10" V 4980 4200 50  0000 C CNN
 F 1 "100" V 4900 4200 50  0000 C CNN
-F 2 "Resistors_SMD:R_0805" V 4830 4200 50  0001 C CNN
+F 2 "rgb-matrix:R_0805" V 4830 4200 50  0001 C CNN
 F 3 "" H 4900 4200 50  0000 C CNN
 	1    4900 4200
@@
 F 0 "R9" V 4980 4100 50  0000 C CNN
 F 1 "100" V 4900 4100 50  0000 C CNN
-F 2 "Resistors_SMD:R_0805" V 4830 4100 50  0001 C CNN
+F 2 "rgb-matrix:R_0805" V 4830 4100 50  0001 C CNN
 F 3 "" H 4900 4100 50  0000 C CNN
 	1    4900 4100
@@
 F 0 "R8" V 4980 4000 50  0000 C CNN
 F 1 "100" V 4900 4000 50  0000 C CNN
-F 2 "Resistors_SMD:R_0805" V 4830 4000 50  0001 C CNN
+F 2 "rgb-matrix:R_0805" V 4830 4000 50  0001 C CNN
 F 3 "" H 4900 4000 50  0000 C CNN
 	1    4900 4000
@@
 F 0 "R7" V 4980 3900 50  0000 C CNN
 F 1 "100" V 4900 3900 50  0000 C CNN
-F 2 "Resistors_SMD:R_0805" V 4830 3900 50  0001 C CNN
+F 2 "rgb-matrix:R_0805" V 4830 3900 50  0001 C CNN
 F 3 "" H 4900 3900 50  0000 C CNN
 	1    4900 3900
@@
 F 0 "R13" V 6630 2900 50  0000 C CNN
 F 1 "100" V 6550 2900 50  0000 C CNN
-F 2 "Resistors_SMD:R_0805" V 6480 2900 50  0001 C CNN
+F 2 "rgb-matrix:R_0805" V 6480 2900 50  0001 C CNN
 F 3 "" H 6550 2900 50  0000 C CNN
 	1    6550 2900
@@
 F 0 "R24" V 6630 4400 50  0000 C CNN
 F 1 "100" V 6550 4400 50  0000 C CNN
-F 2 "Resistors_SMD:R_0805" V 6480 4400 50  0001 C CNN
+F 2 "rgb-matrix:R_0805" V 6480 4400 50  0001 C CNN
 F 3 "" H 6550 4400 50  0000 C CNN
 	1    6550 4400
@@
 F 0 "R23" V 6630 4300 50  0000 C CNN
 F 1 "100" V 6550 4300 50  0000 C CNN
-F 2 "Resistors_SMD:R_0805" V 6480 4300 50  0001 C CNN
+F 2 "rgb-matrix:R_0805" V 6480 4300 50  0001 C CNN
 F 3 "" H 6550 4300 50  0000 C CNN
 	1    6550 4300
@@
 F 0 "R22" V 6630 4200 50  0000 C CNN
 F 1 "100" V 6550 4200 50  0000 C CNN
-F 2 "Resistors_SMD:R_0805" V 6480 4200 50  0001 C CNN
+F 2 "rgb-matrix:R_0805" V 6480 4200 50  0001 C CNN
 F 3 "" H 6550 4200 50  0000 C CNN
 	1    6550 4200
@@
 F 0 "R21" V 6630 4100 50  0000 C CNN
 F 1 "100" V 6550 4100 50  0000 C CNN
-F 2 "Resistors_SMD:R_0805" V 6480 4100 50  0001 C CNN
+F 2 "rgb-matrix:R_0805" V 6480 4100 50  0001 C CNN
 F 3 "" H 6550 4100 50  0000 C CNN
 	1    6550 4100
@@
 F 0 "R20" V 6630 4000 50  0000 C CNN
 F 1 "100" V 6550 4000 50  0000 C CNN
-F 2 "Resistors_SMD:R_0805" V 6480 4000 50  0001 C CNN
+F 2 "rgb-matrix:R_0805" V 6480 4000 50  0001 C CNN
 F 3 "" H 6550 4000 50  0000 C CNN
 	1    6550 4000
@@
 F 0 "R19" V 6630 3900 50  0000 C CNN
 F 1 "100" V 6550 3900 50  0000 C CNN
-F 2 "Resistors_SMD:R_0805" V 6480 3900 50  0001 C CNN
+F 2 "rgb-matrix:R_0805" V 6480 3900 50  0001 C CNN
 F 3 "" H 6550 3900 50  0000 C CNN
 	1    6550 3900
@@
 F 0 "R14" V 6630 3000 50  0000 C CNN
 F 1 "100" V 6550 3000 50  0000 C CNN
-F 2 "Resistors_SMD:R_0805" V 6480 3000 50  0001 C CNN
+F 2 "rgb-matrix:R_0805" V 6480 3000 50  0001 C CNN
 F 3 "" H 6550 3000 50  0000 C CNN
 	1    6550 3000
@@
 F 0 "R15" V 6630 3100 50  0000 C CNN
 F 1 "100" V 6550 3100 50  0000 C CNN
-F 2 "Resistors_SMD:R_0805" V 6480 3100 50  0001 C CNN
+F 2 "rgb-matrix:R_0805" V 6480 3100 50  0001 C CNN
 F 3 "" H 6550 3100 50  0000 C CNN
 	1    6550 3100
@@
 F 0 "R16" V 6630 3200 50  0000 C CNN
 F 1 "100" V 6550 3200 50  0000 C CNN
-F 2 "Resistors_SMD:R_0805" V 6480 3200 50  0001 C CNN
+F 2 "rgb-matrix:R_0805" V 6480 3200 50  0001 C CNN
 F 3 "" H 6550 3200 50  0000 C CNN
 	1    6550 3200
@@
 F 0 "R17" V 6630 3300 50  0000 C CNN
 F 1 "100" V 6550 3300 50  0000 C CNN
-F 2 "Resistors_SMD:R_0805" V 6480 3300 50  0001 C CNN
+F 2 "rgb-matrix:R_0805" V 6480 3300 50  0001 C CNN
 F 3 "" H 6550 3300 50  0000 C CNN
 	1    6550 3300
@@
 F 0 "R18" V 6630 3400 50  0000 C CNN
 F 1 "100" V 6550 3400 50  0000 C CNN
-F 2 "Resistors_SMD:R_0805" V 6480 3400 50  0001 C CNN
+F 2 "rgb-matrix:R_0805" V 6480 3400 50  0001 C CNN
 F 3 "" H 6550 3400 50  0000 C CNN
 	1    6550 3400
