File: hardware/power.sch (KiCad schematic (older format))
At the start: 16 parts, among them CON1 VEXT, P6 VEXT, U6 LD3985M33R

Commit message: Fix silkscreen
Parts:
- C12, C13, C14, C15, C19, C20, C9: footprint Capacitors_SMD:C_0805 -> rgb-matrix:C_0805
- CON1: footprint Connect:BARREL_JACK -> rgb-matrix:BARREL_JACK
- P6: footprint Pin_Headers:Pin_Header_Angled_1x02 -> rgb-matrix:Pin_Header_Angled_1x02
- R28, R29: footprint Resistors_SMD:R_0805 -> rgb-matrix:R_0805
Changed lines of the file:
@@
 F 0 "C9" H 1925 5000 50  0000 L CNN
 F 1 "1uF" H 1925 4800 50  0000 L CNN
-F 2 "Capacitors_SMD:C_0805" H 1938 4750 50  0001 C CNN
+F 2 "rgb-matrix:C_0805" H 1938 4750 50  0001 C CNN
 F 3 "" H 1900 4900 50  0000 C CNN
 	1    1900 4900
@@
 F 0 "C14" H 3325 4950 50  0000 L CNN
 F 1 "1uF" H 3325 4750 50  0000 L CNN
-F 2 "Capacitors_SMD:C_0805" H 3338 4700 50  0001 C CNN
+F 2 "rgb-matrix:C_0805" H 3338 4700 50  0001 C CNN
 F 3 "" H 3300 4850 50  0000 C CNN
 	1    3300 4850
@@
 F 0 "C12" H 2125 5150 50  0000 L CNN
 F 1 "100nF" H 2125 4950 50  0000 L CNN
-F 2 "Capacitors_SMD:C_0805" H 2138 4900 50  0001 C CNN
+F 2 "rgb-matrix:C_0805" H 2138 4900 50  0001 C CNN
 F 3 "" H 2100 5050 50  0000 C CNN
 	1    2100 5050
@@
 F 0 "C13" H 3125 5100 50  0000 L CNN
 F 1 "10nF" H 3125 4900 50  0000 L CNN
-F 2 "Capacitors_SMD:C_0805" H 3138 4850 50  0001 C CNN
+F 2 "rgb-matrix:C_0805" H 3138 4850 50  0001 C CNN
 F 3 "" H 3100 5000 50  0000 C CNN
 	1    3100 5000
@@
 F 0 "C15" H 3575 5150 50  0000 L CNN
 F 1 "100nF" H 3575 4950 50  0000 L CNN
-F 2 "Capacitors_SMD:C_0805" H 3588 4900 50  0001 C CNN
+F 2 "rgb-matrix:C_0805" H 3588 4900 50  0001 C CNN
 F 3 "" H 3550 5050 50  0000 C CNN
 	1    3550 5050
@@
 F 0 "CON1" H 2000 2600 50  0000 C CNN
 F 1 "VEXT" H 2000 2150 50  0000 C CNN
-F 2 "Connect:BARREL_JACK" H 2000 2350 50  0001 C CNN
+F 2 "rgb-matrix:BARREL_JACK" H 2000 2350 50  0001 C CNN
 F 3 "" H 2000 2350 50  0000 C CNN
 	1    2000 2350
@@
 F 0 "P6" H 1750 1800 50  0000 C CNN
 F 1 "VEXT" V 1850 1650 50  0000 C CNN
-F 2 "Pin_Headers:Pin_Header_Angled_1x02" H 1750 1650 50  0001 C CNN
+F 2 "rgb-matrix:Pin_Header_Angled_1x02" H 1750 1650 50  0001 C CNN
 F 3 "" H 1750 1650 50  0000 C CNN
 	1    1750 1650
@@
 F 0 "R29" V 6080 2550 50  0000 C CNN
 F 1 "1k" V 6000 2550 50  0000 C CNN
-F 2 "Resistors_SMD:R_0805" V 5930 2550 50  0001 C CNN
+F 2 "rgb-matrix:R_0805" V 5930 2550 50  0001 C CNN
 F 3 "" H 6000 2550 50  0000 C CNN
 	1    6000 2550
@@
 $EndComp
 $Comp
-L GND #PWR053
+L GND #PWR052
 U 1 1 582B766A
 P 6450 2050
-F 0 "#PWR053" H 6450 1800 50  0001 C CNN
+F 0 "#PWR052" H 6450 1800 50  0001 C CNN
 F 1 "GND" H 6450 1900 50  0000 C CNN
 F 2 "" H 6450 2050 50  0000 C CNN
@@
 F 0 "R28" V 6080 2050 50  0000 C CNN
 F 1 "1k" V 6000 2050 50  0000 C CNN
-F 2 "Resistors_SMD:R_0805" V 5930 2050 50  0001 C CNN
+F 2 "rgb-matrix:R_0805" V 5930 2050 50  0001 C CNN
 F 3 "" H 6000 2050 50  0000 C CNN
 	1    6000 2050
@@
 $EndComp
 $Comp
-L +3V3 #PWR054
+L +3V3 #PWR053
 U 1 1 582B7677
 P 5750 2050
-F 0 "#PWR054" H 5750 1900 50  0001 C CNN
+F 0 "#PWR053" H 5750 1900 50  0001 C CNN
 F 1 "+3V3" H 5750 2190 50  0000 C CNN
 F 2 "" H 5750 2050 50  0000 C CNN
@@
 $EndComp
 $Comp
-L GND #PWR055
+L GND #PWR054
 U 1 1 582B7858
 P 4450 4900
-F 0 "#PWR055" H 4450 4650 50  0001 C CNN
+F 0 "#PWR054" H 4450 4650 50  0001 C CNN
 F 1 "GND" H 4450 4750 50  0000 C CNN
 F 2 "" H 4450 4900 50  0000 C CNN
@@
 $EndComp
 $Comp
-L PWR_FLAG #FLG056
+L PWR_FLAG #FLG055
 U 1 1 582B785E
 P 4450 4800
-F 0 "#FLG056" H 4450 4895 50  0001 C CNN
+F 0 "#FLG055" H 4450 4895 50  0001 C CNN
 F 1 "PWR_FLAG" H 4450 4980 50  0000 C CNN
 F 2 "" H 4450 4800 50  0000 C CNN
@@
 $EndComp
 $Comp
-L +5V #PWR057
+L +5V #PWR056
 U 1 1 582B7864
 P 4850 4750
-F 0 "#PWR057" H 4850 4600 50  0001 C CNN
+F 0 "#PWR056" H 4850 4600 50  0001 C CNN
 F 1 "+5V" H 4850 4890 50  0000 C CNN
 F 2 "" H 4850 4750 50  0000 C CNN
@@
 $EndComp
 $Comp
-L PWR_FLAG #FLG058
+L PWR_FLAG #FLG057
 U 1 1 582B786A
 P 4850 4850
-F 0 "#FLG058" H 4850 4945 50  0001 C CNN
+F 0 "#FLG057" H 4850 4945 50  0001 C CNN
 F 1 "PWR_FLAG" H 4850 5030 50  0000 C CNN
 F 2 "" H 4850 4850 50  0000 C CNN
@@
 VEXT
 $Comp
-L +5V #PWR059
+L +5V #PWR058
 U 1 1 58729962
 P 4650 1900
-F 0 "#PWR059" H 4650 1750 50  0001 C CNN
+F 0 "#PWR058" H 4650 1750 50  0001 C CNN
 F 1 "+5V" H 4650 2040 50  0000 C CNN
 F 2 "" H 4650 1900 50  0000 C CNN
@@
 F 0 "C19" H 2925 2550 50  0000 L CNN
 F 1 "10uF" H 2925 2350 50  0000 L CNN
-F 2 "Capacitors_SMD:C_0805" H 2938 2300 50  0001 C CNN
+F 2 "rgb-matrix:C_0805" H 2938 2300 50  0001 C CNN
 F 3 "" H 2900 2450 50  0000 C CNN
 	1    2900 2450
@@
 $EndComp
 $Comp
-L GND #PWR060
+L GND #PWR059
 U 1 1 5873D009
 P 2900 2600
-F 0 "#PWR060" H 2900 2350 50  0001 C CNN
+F 0 "#PWR059" H 2900 2350 50  0001 C CNN
 F 1 "GND" H 2900 2450 50  0000 C CNN
 F 2 "" H 2900 2600 50  0000 C CNN
@@
 F 0 "C20" H 2925 3250 50  0000 L CNN
 F 1 "10uF" H 2925 3050 50  0000 L CNN
-F 2 "Capacitors_SMD:C_0805" H 2938 3000 50  0001 C CNN
+F 2 "rgb-matrix:C_0805" H 2938 3000 50  0001 C CNN
 F 3 "" H 2900 3150 50  0000 C CNN
 	1    2900 3150
@@
 $EndComp
 $Comp
-L GND #PWR061
+L GND #PWR060
 U 1 1 5873D127
 P 2900 3300
-F 0 "#PWR061" H 2900 3050 50  0001 C CNN
+F 0 "#PWR060" H 2900 3050 50  0001 C CNN
 F 1 "GND" H 2900 3150 50  0000 C CNN
 F 2 "" H 2900 3300 50  0000 C CNN
@@
 $EndComp
 $Comp
-L VCC #PWR062
+L VCC #PWR061
 U 1 1 587478CE
 P 5750 4750
-F 0 "#PWR062" H 5750 4600 50  0001 C CNN
+F 0 "#PWR061" H 5750 4600 50  0001 C CNN
 F 1 "VCC" H 5750 4900 50  0000 C CNN
 F 2 "" H 5750 4750 50  0000 C CNN
@@
 $EndComp
 Wire Wire Line
-	1950 2950 2900 2950
-Wire Wire Line
-	2900 2950 3650 2950
+	1950 2950 3650 2950
 Wire Wire Line
 	4450 4800 4450 4900
@@
 	2300 1700 1950 1700
 Wire Wire Line
-	2300 2250 2400 2250
-Wire Wire Line
-	2400 2250 2900 2250
-Wire Wire Line
-	2900 2250 3650 2250
+	2300 2250 3650 2250
 Connection ~ 2300 2450
 Wire Wire Line
-	2300 2350 2300 2450
-Wire Wire Line
-	2300 2450 2300 2550
+	2300 2350 2300 2550
 Connection ~ 3550 4650
 Wire Wire Line
@@
 Connection ~ 1900 5200
 Wire Wire Line
-	1900 5200 2100 5200
-Wire Wire Line
-	2100 5200 2650 5200
-Wire Wire Line
-	2650 5200 3100 5200
-Wire Wire Line
-	3100 5200 3300 5200
-Wire Wire Line
-	3300 5200 3550 5200
+	1900 5200 3550 5200
 Connection ~ 2100 4800
 Connection ~ 1900 4650
 Connection ~ 2100 4650
 Wire Wire Line
-	2100 4650 2100 4800
-Wire Wire Line
-	2100 4800 2100 4900
+	2100 4650 2100 4900
 Wire Wire Line
 	2200 4800 2100 4800
 Wire Wire Line
-	3100 4650 3300 4650
-Wire Wire Line
-	3300 4650 3550 4650
-Wire Wire Line
-	1900 4650 2100 4650
-Wire Wire Line
-	2100 4650 2200 4650
-Wire Wire Line
-	1900 4600 1900 4650
-Wire Wire Line
-	1900 4650 1900 4750
-Wire Wire Line
-	3550 4500 3550 4650
-Wire Wire Line
-	3550 4650 3550 4900
+	3100 4650 3550 4650
+Wire Wire Line
+	1900 4650 2200 4650
+Wire Wire Line
+	1900 4600 1900 4750
+Wire Wire Line
+	3550 4500 3550 4900
 Wire Wire Line
 	3300 5200 3300 5000
 Wire Wire Line
-	1900 5050 1900 5200
-Wire Wire Line
-	1900 5200 1900 5250
+	1900 5050 1900 5250
 Wire Wire Line
 	2900 2300 2900 2250
@@
 	5250 4750 5250 5000
 Wire Wire Line
-	5250 5000 5500 5000
-Wire Wire Line
-	5500 5000 5750 5000
+	5250 5000 5750 5000
 Connection ~ 5500 5000
 $Comp
@@
 	4250 2250 4650 2250
 Wire Wire Line
-	4650 1900 4650 2250
-Wire Wire Line
-	4650 2250 4650 2950
+	4650 1900 4650 2950
 Wire Wire Line
 	4650 2950 4250 2950
@@
 	5750 2550 5850 2550
 $Comp
-L +5V #PWR?
+L +5V #PWR062
 U 1 1 58800ECC
 P 5750 2550
-F 0 "#PWR?" H 5750 2400 50  0001 C CNN
+F 0 "#PWR062" H 5750 2400 50  0001 C CNN
 F 1 "+5V" H 5750 2690 50  0000 C CNN
 F 2 "" H 5750 2550 50  0000 C CNN

Commit message: Add 2nd GND pin for more curent + minor changes
Parts:
- P6: footprint rgb-matrix:Pin_Header_Angled_1x02 -> Pin_Headers:Pin_Header_Straight_1x02_Pitch2.54mm
Changed lines of the file:
@@
 F 0 "P6" H 1750 1800 50  0000 C CNN
 F 1 "VEXT" V 1850 1650 50  0000 C CNN
-F 2 "rgb-matrix:Pin_Header_Angled_1x02" H 1750 1650 50  0001 C CNN
+F 2 "Pin_Headers:Pin_Header_Straight_1x02_Pitch2.54mm" H 1750 1650 50  0001 C CNN
 F 3 "" H 1750 1650 50  0000 C CNN
 	1    1750 1650
@@
 Wire Wire Line
 	2300 1700 2300 1750
-Connection ~ 2400 2250
-Wire Wire Line
-	2400 1600 2400 2250
 Wire Wire Line
 	1950 1600 2400 1600
@@
 	0    -1   -1   0
 $EndComp
+Connection ~ 2400 2250
+Wire Wire Line
+	2400 1600 2400 2250
 $EndSCHEMATC
